File: SunnyBuddyv10/SunnyBuddy.brd (EAGLE design)
At the start: 47 x 47 mm, 35 parts, among them J1 5.5x2.1mm Barrel, J3 POWER_JACKPTH, J5 M02PTH, J6 M023.5MM, J7 M023.5MM, J8 M023.5MM, U1 LT3652

Commit message: commit
Parts:
- removed C1: 10uF, SparkFun-Capacitors:1210
- removed C2: 10uF, SparkFun-Capacitors:1206
- removed C3, C4: 47uF, SparkFun-Capacitors:EIA3528
- removed C5, C6: 1.0uF, SparkFun-Capacitors:0603-CAP
- removed D1, D2: ZLLS500, SparkFun-DiscreteSemi:SOT23
- removed FID1, FID2: FIDUCIAL1X2, SparkFun-Aesthetics:FIDUCIAL-1X2
- removed J4: (no value), SparkFun-Connectors:JST-2-SMD
- removed L1: 68uH, SparkFun-Passives:CR75
- removed LOGO1: SFE_LOGO_NAME_FLAME.2_INCH, SparkFun-Aesthetics:SFE_LOGO_NAME_FLAME_.2
- removed LOGO2: OSHW-LOGOM, SparkFun-Aesthetics:OSHW-LOGO-M
- removed R1: 0.22, SparkFun-Resistors:0805
- removed R2: 100k, SparkFun-Resistors:0603-RES
- removed R3: 300k, SparkFun-Resistors:0603-RES
- removed R6: 0, SparkFun-Resistors:0603
- removed U1: LT3652, SparkFun-PowerIC:MSOP-12_GND
Connections:
- removed net BOOST: C5.1, D2.3, U1.11
- removed net FB: R2.1, R3.2, R6.2
- removed net N$3: R6.1, U1.7
- removed net NTC: U1.8
- removed net SENSE: L1.P$2, R1.1, U1.10
- removed net SW: C5.2, D1.3, L1.P$1, U1.12
- removed net TIMER: C6.2, U1.6
- net !CHRG: no longer U1.4
- net !FAULT: no longer U1.5
- net GND: no longer C1.2, C2.2, C3.C, C4.C, C6.1, D1.1, J4.1, J4.NC1, J4.NC2, R3.1, U1.13
- net VIN: no longer C1.1, U1.1, U1.2, U1.3
- net V_BATT: no longer C2.1, C3.A, C4.A, D2.1, J4.2, R1.2, R2.2, U1.9
Routing:
- net SENSE: track 24.7 -> 0.00 mm, vias 2 -> 0
- net V_BATT: track 85.1 -> 64.1 mm
- net VIN: track 23.5 -> 8.11 mm
- net GND: track 8.51 -> 2.16 mm
- net BOOST: track 5.83 -> 0.00 mm
- net SW: track 5.28 -> 0.00 mm
- net N$3: track 4.10 -> 0.00 mm
- net FB: track 3.25 -> 0.00 mm
- net !FAULT: track 36.1 -> 34.0 mm
- net TIMER: track 1.89 -> 0.00 mm
- net !CHRG: track 32.5 -> 31.0 mm
