File: SunnyBuddyv10/SunnyBuddy.sch (EAGLE design)
At the start: 35 parts, among them J1 5.5x2.1mm Barrel, J3 POWER_JACKPTH, J5 M02PTH, J6 M023.5MM, J7 M023.5MM, J8 M023.5MM, U1 LT3652

Commit message: commit
Parts:
- removed C1: 10uF, SparkFun-Capacitors:10UF50V20%(1210)
- removed C2: 10uF, SparkFun-Capacitors:10UF-6.3V-20%(1206)
- removed C3, C4: 47uF, SparkFun-Capacitors:47UF-TANT
- removed C5, C6: 1.0uF, SparkFun-Capacitors:1.0UF-16V-10%(0603)
- removed D1, D2: ZLLS500, SparkFun-DiscreteSemi:ZLLS500ZLLS500
- removed FID1, FID2: FIDUCIAL1X2, SparkFun-Aesthetics:FIDUCIAL1X2
- removed J4: (no value), SparkFun-Connectors:JST_2MM_MALE
- removed L1: 68uH, SparkFun-Passives:INDUCTOR68UH-1A
- removed LOGO1: SFE_LOGO_NAME_FLAME.2_INCH, SparkFun-Aesthetics:SFE_LOGO_NAME_FLAME.2_INCH
- removed LOGO2: OSHW-LOGOM, SparkFun-Aesthetics:OSHW-LOGOM
- removed R1: 0.22, SparkFun-Resistors:0.22OHM1/4W1%(0805)
- removed R2: 100k, SparkFun-Resistors:100KOHM1/10W1%(0603)
- removed R3: 300k, SparkFun-Resistors:300KOHM-1/10W-1%(0603)
- removed R6: 0, SparkFun-Resistors:0OHM1/10W5%(0603)
- removed U1: LT3652, SparkFun-PowerIC:LT3652
Connections:
- removed net BOOST: C5.1, D2.C, U1.BOOST
- removed net FB: R2.1, R3.2, R6.2
- removed net N$3: R6.1, U1.VFB
- removed net NTC: U1.NTC
- removed net SENSE: L1.2, R1.1, U1.SENSE
- removed net SW: C5.2, D1.C, L1.1, U1.SW
- removed net TIMER: C6.2, U1.TIMER
- net !CHRG: no longer U1.!CHRG
- net !FAULT: no longer U1.!FAULT
- net GND: no longer C1.2, C2.2, C3.-, C4.-, C6.1, D1.A, J4.-, J4.PAD1, J4.PAD2, R3.1, U1.GND_PAD
- net VIN: no longer C1.1, U1.!SHDN, U1.VIN, U1.VIN_REG
- net V_BATT: no longer C2.1, C3.+, C4.+, D2.A, J4.+, R1.2, R2.2, U1.BAT
Other:
- note removed: "M. Hord"
- note removed: "NB: With both JP1 and JP2 shorted, the second power input is also shorted! You've been warned!"
- note removed: "To add a second bank of solar cells, short JP2 and clear JP1."
