File: SunnyBuddy-v13 2/SunnyBuddy-v13.sch (EAGLE design)
At the start: 35 parts, among them J1 5.5x2.1mm Barrel, J3 POWER_JACKPTH, J5 M02PTH, J6 M023.5MM, J7 M023.5MM, J8 M023.5MM, U1 LT3652

Commit message: sunny
Parts:
- added J2: POWER_JACKPTH, SparkFun-Connectors:POWER_JACKPTH
- added JP4: R_SEN, SparkFun-Connectors:M02PTH
- added LOGO3: OSHW-LOGOS, SparkFun-Aesthetics:OSHW-LOGOS
- added LOGO4: SFE_LOGO_NAME_FLAME.3_INCH, SparkFun-Aesthetics:SFE_LOGO_NAME_FLAME.3_INCH
- added R7: 10k, SparkFun-Electromechanical:TRIMPOTRES-09285
- J3: value POWER_JACKPTH -> (none); device SparkFun-Connectors:POWER_JACKPTH -> SparkFun-Connectors:JST_2MM_MALE
- J4: device SparkFun-Connectors:JST_2MM_MALE -> SparkFun-Connectors:M04PTH
- JP3: value (none) -> JUMPER-PTH-2-NC; device SparkFun-Connectors:M03PTH -> SparkFun-Passives:JUMPER-PTH-2-NC
- R2: value 100k -> 47k; device SparkFun-Resistors:100KOHM1/10W1%(0603) -> SparkFun-Resistors:47KOHM1/10W1%(0603)
- R3: value 300k -> 220k; device SparkFun-Resistors:300KOHM-1/10W-1%(0603) -> SparkFun-Resistors:220KOHM1/10W1%(0603)
- R6: value 0 -> 220k; device SparkFun-Resistors:0OHM1/10W5%(0603) -> SparkFun-Resistors:220KOHM1/10W1%(0603)
Connections:
- new net N$4: C2.1, C3.+, C4.+, D2.A, JP3.1, JP4.1, R1.2, R2.2, U1.BAT
- new net SET: J4.4, R7.WIPER, U1.VIN_REG
- net !CHRG: now also J4.1; no longer JP3.1
- net !FAULT: now also J4.2; no longer JP3.2
- net GND: now also J3.-, J3.PAD1, J3.PAD2, J4.3, R7.CW; no longer J4.-, J4.PAD1, J4.PAD2, JP3.3
- net N$8: now also J2.GND, J2.GNDBREAK; no longer J3.GND, J3.GNDBREAK
- net SENSE: now also JP4.2
- net SFSASDF: now also J2.PWR; no longer J3.PWR
- net VIN: now also R7.CCW; no longer U1.VIN_REG
- net V_BATT: now also J3.+, JP3.2; no longer C2.1, C3.+, C4.+, D2.A, J4.+, R1.2, R2.2, U1.BAT
Other:
- note added: "0.22 -> 800mA"
- note added: "0.33 -> 750mA"
- note added: "0.5 -> 650mA"
- note added: "1.0 -> 550mA"
- note added: "Cut the JP3 trace to measure output current. Adjust trim pot until output current reaches its maximum."
- note added: "Ichg = .1/(R1||Rsen)"
- note added: "NB: With both JP1 and JP2 shorted, the second power input is also shorted! This may result in damage to your power source. You've been warned!"
- note added: "R_SEN is in parallel with R1. Small resistors can be added to increase the charge current from the default ~450mA."
- note added: "Typical R_SEN values vs. Ichg"
- note added: "Voltage at SET can be used to set MPPT level. In full sun, adjust pot until V_SET = 2.8V."
- note added: "v13"
- note removed: "NB: With both JP1 and JP2 shorted, the second power input is also shorted! You've been warned!"
- note removed: "v10"
- moved on the sheet: C1, D1
